Commit message: backup,may have bugs

File: src/sentry_simulation/urdf/livox_mid360.urdf.xacro (robot description, xacro)
@@ -1,5 +1,5 @@
 <robot name="livox_base" xmlns:xacro="http://www.ros.org/wiki/xacro">
   <xacro:property name="PI" value="3.1415926"/>
-  <xacro:property name="visualize" value="true" />
+  <xacro:property name="visualize" value="false" />
   <xacro:property name="update_rate" value="10" />
   <xacro:property name="resolution" value="0.002" />
@@ -41,5 +41,5 @@
   </link>
   <joint name="livox_mid360_joint" type="fixed">
-    <origin xyz="0 0 0.31" rpy="0 0 0" />
+    <origin xyz="0 0 0.25" rpy="0 0 0" />
     <parent link="base_link" />
     <child link="livox_mid360" />
